File: pcbs/lablogger_board/lablogger_board.kicad_sch (KiCad schematic)
At the start: 45 parts, among them J10 5mm, J11 DB9, J12 DB9, J2 Conn_01x07, J3 Conn_01x12, J4 PINHD-1X4, J5 5mm, J6 5mm, J7 RJ11, J8 RJ11, J9 5mm, P1 24V / 5A, Q3 220mA / 50V, Q4 220mA / 50V, Q5 5.7A / 30V, Q6 5.7A / 30V, U1 8-28V in / 5V 5W out, U2 Particle2 / Boron, U3 RS485 Transceiver, U4 RS232 Transceiver

Commit message: lablogger first version
Parts:
- C5: JLCPCB (none) -> C1591; JLCPCBURL (none) -> https://jlcpcb.com/partdetail/1943-CL10B104KB8NNNC/C1591
- F1: footprint footprints:Fuse_1812 -> footprints:Fuse_2920_7451
- J5: footprint footprints:TERMINAL_BLOCK_1x02V_5mm -> footprints:TERMINAL_BLOCK_1x02_5mm_vertical
- R11: JLCPCB (none) -> C17902; JLCPCBURL (none) -> https://jlcpcb.com/partdetail/18590-1206W4F1002T5E/C17902
- renumbered D2 to D1, D1 to D2, Q5 to Q1, Q6 to Q2, R22 to R10, R23 to R15, R7 to R3, R17 to R4, R16 to R5, R19 to R6, R15 to R7, R20 to R8, R21 to R9
Connections:
- net D17-1Wire: now also J9.2, R10.2
- removed net D6-1Wire: J9.2, R10.2, U2.23 (D6)
- new net D6: U2.23 (D6)
- no-connect marks 20 -> 21
